File: Vector.kicad_pcb (KiCad board)
At the start: 2 copper layers, 54.6 x 52.7 mm, 37 parts, among them J1 Conn_01x06_Female, J2 Barrel_Jack_Switch, Q1 BC547, Q2 BC547, Q3 BC547, Q4 BC547

Commit message: Migrate to KiCAD 6
Other:
- net class Default removed

Commit message: Update symbols/footprints from libraries
Parts:
- R11: value 390k -> 22k
- R12: value 470k -> 100k
- moved RV1 5.04 mm to (99.7, 60.3)
- moved RV2 5.04 mm to (126.4, 60.3)
Connections:
- J1 pad 2: Net-(J1-Pad2) -> unconnected-(J1-Pad2)
- RV1 pad 1: Net-(R11-Pad2) -> Net-(R10-Pad1)
- RV1 pad 3: Net-(R10-Pad1) -> Net-(R11-Pad2)
- RV2 pad 1: Net-(C8-Pad1) -> GND
- RV2 pad 3: GND -> Net-(C8-Pad1)
