File: Vector.kicad_sch (KiCad schematic)
At the start: 33 parts

Commit message: Update symbols/footprints from libraries
Parts:
- C1, C3, C5, C6, C7: value (none) -> 100n; footprint (none) -> Capacitor_THT:C_Rect_L7.2mm_W2.5mm_P5.00mm_FKS2_FKP2_MKS2_MKP2
- C2, C8: value (none) -> 1µ; footprint (none) -> Capacitor_THT:C_Rect_L7.2mm_W4.5mm_P5.00mm_FKS2_FKP2_MKS2_MKP2
- C4: value (none) -> 470n; footprint (none) -> Capacitor_THT:C_Rect_L7.2mm_W3.5mm_P5.00mm_FKS2_FKP2_MKS2_MKP2
- D1, D2: value (none) -> 1N4148; footprint (none) -> Diode_THT:D_DO-35_SOD27_P2.54mm_Vertical_AnodeUp
- J1: value (none) -> Conn_01x06_Female; footprint (none) -> Connector_PinHeader_2.54mm:PinHeader_1x06_P2.54mm_Vertical
- J2: value (none) -> Barrel_Jack_Switch; footprint (none) -> NLS:BarrelJack_Horizontal_Short
- Q1, Q2, Q3, Q4: value (none) -> BC547; footprint (none) -> Package_TO_SOT_THT:TO-92_Wide
- R1, R13, R2, R5: value (none) -> 1M; footprint (none) -> Resistor_THT:R_Axial_DIN0207_L6.3mm_D2.5mm_P2.54mm_Vertical
- R10: value (none) -> 470k; footprint (none) -> Resistor_THT:R_Axial_DIN0207_L6.3mm_D2.5mm_P7.62mm_Horizontal
- R11: value (none) -> 22k; footprint (none) -> Resistor_THT:R_Axial_DIN0207_L6.3mm_D2.5mm_P7.62mm_Horizontal
- R12: value (none) -> 100k; footprint (none) -> Resistor_THT:R_Axial_DIN0207_L6.3mm_D2.5mm_P7.62mm_Horizontal
- R14, R3: value (none) -> 10k; footprint (none) -> Resistor_THT:R_Axial_DIN0207_L6.3mm_D2.5mm_P2.54mm_Vertical
- R15: value (none) -> 39k; footprint (none) -> Resistor_THT:R_Axial_DIN0207_L6.3mm_D2.5mm_P7.62mm_Horizontal
- R4, R7, R8, R9: value (none) -> 100k; footprint (none) -> Resistor_THT:R_Axial_DIN0207_L6.3mm_D2.5mm_P2.54mm_Vertical
- R6: value (none) -> 470k; footprint (none) -> Resistor_THT:R_Axial_DIN0207_L6.3mm_D2.5mm_P2.54mm_Vertical
- RV1: value (none) -> 100k; footprint (none) -> Potentiometer_THT:Potentiometer_Alps_RK09K_Single_Vertical; symbol Vector-rescue:R_POT-Device -> Device:R_Potentiometer
Connections:
- net GND: now also RV2.1; no longer RV2.3
- net at R11.2, R9.2: now also RV1.3; no longer RV1.1
- net at C8.1: now also RV2.3; no longer RV2.1
- net at R10.1, R12.2: now also RV1.1; no longer RV1.3
